File: GuMStick.kicad_sch (KiCad schematic)
At the start: 35 parts, among them Q1 SI2302, Q2 SI2302, SW1 K3-1235S, SW2 K3-1235S, U1 XIAO-nRF52840-SMD, U2 Wio-SX1262, U3 M20-7910442R, U5 BQ25606RGER

Commit message: PCB updated to include reverse polarity protection via MOSFET, added diode to battery pin on XIAO to allow battery voltage detection without allowing charging.
Parts:
- added D4: 1N5819WS, Diode_SMD:D_SOD-323, symbol Diode:1N5819WS
Connections:
- net BAT+: now also D4.2 (A)
- net at U1.32 (BAT): now also D4.1 (K)
- no-connect marks 14 -> 13

Commit message: Removed 180R on buzzer
Parts:
- removed R1: 180Ω, PCM_JLCPCB:R_0603, symbol PCM_JLCPCB-Resistors:0603,180Ω
- D4: LCSC Part (none) -> C191023; MPN (none) -> 1N5819WS
- L1: LCSC C1042 -> C5339212; MPN SDFL2012Q1R0KTF -> YWLD2012-1R0K; Manufacturer Sunlord -> YJYCOIN; Minimum Qty 20 -> 10; Part SDFL2012Q1R0KTF -> YWLD2012-1R0K; Price 0.020USD -> 0.063USD; Rated Current 50mA -> 1A
Connections:
- net BUZ_PWM: now also Q1.1 (G)

Commit message: Fixes to part numbers and details
Parts:
- BAT+1, BAT-1: now not fitted
- D4: footprint Diode_SMD:D_SOD-323 -> easyeda2kicad:SOD-323_L1.8-W1.3-LS2.5-RD; symbol Diode:1N5819WS -> easyeda2kicad:1N5819WS; Manufacturer (none) -> Hottech(合科泰)
- L1: value 1uH,50mA -> 1uH,1A
- Q1, Q2: footprint Package_TO_SOT_SMD:SOT-23 -> easyeda2kicad:SOT-23_L2.9-W1.3-P1.90-LS2.4-BR; symbol OPL_Discrete_Semiconductor:SMD-MOSFET-N-CH-20V-2.1A-CJ2302_SOT-23_ -> easyeda2kicad:Si2302CDS-T1-GE3; LCSC Part (none) -> C10488; MPN SI2302CDS-T1-GE3 -> Si2302CDS-T1-GE3; Manufacturer Vishay -> VISHAY(威世)
Changed lines of the file:
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@@
 	(wire
 		(pts
-			(xy 74.93 184.15) (xy 74.93 181.61)
+			(xy 74.93 184.15) (xy 74.93 182.88)
 		)
 		(stroke
@@
 	(wire
 		(pts
-			(xy 116.84 87.63) (xy 119.38 87.63)
+			(xy 116.84 88.9) (xy 119.38 88.9)
 		)
 		(stroke
@@
 	(wire
 		(pts
-			(xy 74.93 167.64) (xy 74.93 173.99)
+			(xy 74.93 167.64) (xy 74.93 172.72)
 		)
 		(stroke
@@
 	(wire
 		(pts
-			(xy 99.06 71.12) (xy 115.57 71.12)
+			(xy 101.6 71.12) (xy 115.57 71.12)
 		)
 		(stroke
@@
 	(wire
 		(pts
-			(xy 132.08 87.63) (xy 129.54 87.63)
+			(xy 132.08 88.9) (xy 129.54 88.9)
 		)
 		(stroke
@@
 	(wire
 		(pts
-			(xy 254 43.18) (xy 254 49.53)
+			(xy 124.46 81.28) (xy 124.46 80.01)
 		)
 		(stroke
@@
 	(wire
 		(pts
-			(xy 254 43.18) (xy 257.81 43.18)
+			(xy 254 43.18) (xy 254 49.53)
 		)
 		(stroke
@@
 	(wire
 		(pts
-			(xy 173.99 111.76) (xy 173.99 110.49)
+			(xy 254 43.18) (xy 257.81 43.18)
 		)
 		(stroke
@@
 	(wire
 		(pts
-			(xy 114.3 121.92) (xy 118.11 121.92)
+			(xy 173.99 111.76) (xy 173.99 110.49)
 		)
 		(stroke
@@
 	(wire
 		(pts
-			(xy 236.22 45.72) (xy 234.95 45.72)
+			(xy 114.3 121.92) (xy 118.11 121.92)
 		)
 		(stroke
@@
 	(wire
 		(pts
-			(xy 124.46 80.01) (xy 124.46 82.55)
+			(xy 236.22 45.72) (xy 234.95 45.72)
 		)
 		(stroke
@@
 	(global_label "RPP S"
 		(shape input)
-		(at 132.08 87.63 0)
+		(at 132.08 88.9 0)
 		(fields_autoplaced yes)
 		(effects
@@
 		)
 		(property "Intersheetrefs" "${INTERSHEET_REFS}"
-			(at 141.0523 87.63 0)
+			(at 141.0523 88.9 0)
 			(hide yes)
 			(show_name no)
@@
 	(global_label "BAT+"
 		(shape input)
-		(at 116.84 87.63 180)
+		(at 116.84 88.9 180)
 		(fields_autoplaced yes)
 		(effects
@@
 		)
 		(property "Intersheetrefs" "${INTERSHEET_REFS}"
-			(at 108.9562 87.63 0)
+			(at 108.9562 88.9 0)
 			(hide yes)
 			(show_name no)
@@
 	)
 	(symbol
-		(lib_id "Diode:1N5819WS")
+		(lib_id "easyeda2kicad:1N5819WS")
 		(at 74.93 177.8 270)
 		(unit 1)
@@
 		(fields_autoplaced yes)
 		(property "Reference" "D4"
-			(at 77.47 176.2124 90)
+			(at 78.74 176.2749 90)
 			(show_name no)
 			(do_not_autoplace no)
@@
 		)
 		(property "Value" "1N5819WS"
-			(at 77.47 178.7524 90)
+			(at 78.74 178.8149 90)
 			(show_name no)
 			(do_not_autoplace no)
@@
 			)
 		)
-		(property "Footprint" "Diode_SMD:D_SOD-323"
-			(at 70.485 177.8 0)
+		(property "Footprint" "easyeda2kicad:SOD-323_L1.8-W1.3-LS2.5-RD"
+			(at 67.31 177.8 0)
 			(hide yes)
 			(show_name no)
@@
 			)
 		)
-		(property "Datasheet" "https://datasheet.lcsc.com/lcsc/2204281430_Guangdong-Hottech-1N5819WS_C191023.pdf"
-			(at 74.93 177.8 0)
+		(property "Datasheet" "https://lcsc.com/product-detail/Others_B5819WS_C191023.html"
+			(at 64.77 177.8 0)
 			(hide yes)
 			(show_name no)
@@
 		)
 		(property "MPN" "1N5819WS"
-			(at 74.93 177.8 90)
+			(at 59.69 177.8 0)
 			(hide yes)
 			(show_name no)
@@
 		)
 		(property "LCSC Part" "C191023"
-			(at 74.93 177.8 90)
+			(at 57.15 177.8 0)
+			(hide yes)
+			(show_name no)
+			(do_not_autoplace no)
+			(effects
+				(font
+					(size 1.27 1.27)
+				)
+			)
+		)
+		(property "Manufacturer" "Hottech(合科泰)"
+			(at 62.23 177.8 0)
 			(hide yes)
 			(show_name no)
@@
 		(on_board yes)
 		(in_pos_files yes)
-		(dnp no)
+		(dnp yes)
 		(property "Reference" "BAT+1"
 			(at 71.374 94.488 0)
@@
 	)
 	(symbol
-		(lib_id "OPL_Discrete_Semiconductor:SMD-MOSFET-N-CH-20V-2.1A-CJ2302_SOT-23_")
-		(at 124.46 87.63 90)
+		(lib_id "easyeda2kicad:Si2302CDS-T1-GE3")
+		(at 124.46 86.36 90)
 		(mirror x)
 		(unit 1)
@@
 		(fields_autoplaced yes)
 		(property "Reference" "Q2"
-			(at 124.6251 92.71 90)
+			(at 124.46 95.25 90)
 			(show_name no)
 			(do_not_autoplace no)
@@
 		)
 		(property "Value" "SI2302"
-			(at 124.6251 95.25 90)
+			(at 124.46 97.79 90)
 			(show_name no)
 			(do_not_autoplace no)
@@
 			)
 		)
-		(property "Footprint" "Package_TO_SOT_SMD:SOT-23"
-			(at 124.46 87.63 0)
+		(property "Footprint" "easyeda2kicad:SOT-23_L2.9-W1.3-P1.90-LS2.4-BR"
+			(at 137.16 86.36 0)
 			(hide yes)
 			(show_name no)
@@
 			)
 		)
-		(property "Datasheet" "https://www.vishay.com/docs/68645/si2302cds.pdf"
-			(at 124.46 87.63 0)
+		(property "Datasheet" "https://lcsc.com/product-detail/MOSFET_VISHAY_Si2302CDS-T1-GE3_Si2302CDS-T1-GE3_C10488.html"
+			(at 139.7 86.36 0)
 			(hide yes)
 			(show_name no)
@@
 			)
 		)
-		(property "Description" "MOSFETs 20V Vds 8V Vgs SOT-23"
-			(at 124.46 87.63 0)
+		(property "Description" "Si2302CDS-T1-GE3"
+			(at 124.46 86.36 0)
 			(hide yes)
 			(show_name no)
@@
 			)
 		)
-		(property "MPN" "SI2302CDS-T1-GE3 "
-			(at 120.65 88.392 0)
+		(property "MPN" "Si2302CDS-T1-GE3"
+			(at 144.78 86.36 0)
 			(hide yes)
 			(show_name no)
@@
 			(effects
 				(font
-					(size 0.508 0.508)
+					(size 1.27 1.27)
 				)
 			)
 		)
-		(property "Manufacturer" "Vishay"
-			(at 124.46 87.63 0)
+		(property "Manufacturer" "VISHAY(威世)"
+			(at 142.24 86.36 0)
+			(hide yes)
+			(show_name no)
+			(do_not_autoplace no)
+			(effects
+				(font
+					(size 1.27 1.27)
+				)
+			)
+		)
+		(property "LCSC Part" "C10488"
+			(at 147.32 86.36 0)
 			(hide yes)
 			(show_name no)
@@
 			)
 		)
-		(property "Value" "1uH,50mA"
+		(property "Value" "1uH,1A"
 			(at 248.666 46.99 90)
 			(show_name no)
@@
 	)
 	(symbol
-		(lib_id "OPL_Discrete_Semiconductor:SMD-MOSFET-N-CH-20V-2.1A-CJ2302_SOT-23_")
-		(at 93.98 71.12 0)
+		(lib_id "easyeda2kicad:Si2302CDS-T1-GE3")
+		(at 96.52 71.12 0)
 		(mirror y)
 		(unit 1)
@@
 		(fields_autoplaced yes)
 		(property "Reference" "Q1"
-			(at 90.17 70.015 0)
+			(at 88.9 69.8499 0)
 			(show_name no)
 			(do_not_autoplace no)
@@
 		)
 		(property "Value" "SI2302"
-			(at 90.17 72.555 0)
+			(at 88.9 72.3899 0)
 			(show_name no)
 			(do_not_autoplace no)
@@
 			)
 		)
-		(property "Footprint" "Package_TO_SOT_SMD:SOT-23"
-			(at 93.98 71.12 0)
+		(property "Footprint" "easyeda2kicad:SOT-23_L2.9-W1.3-P1.90-LS2.4-BR"
+			(at 96.52 83.82 0)
+			(hide yes)
+			(show_name no)
+			(do_not_autoplace no)
+			(effects
+				(font
+					(size 1.27 1.27)
+				)
+			)
+		)
+		(property "Datasheet" "https://lcsc.com/product-detail/MOSFET_VISHAY_Si2302CDS-T1-GE3_Si2302CDS-T1-GE3_C10488.html"
+			(at 96.52 86.36 0)
 			(hide yes)
 			(show_name no)
@@
 			)
 		)
-		(property "Datasheet" "https://www.vishay.com/docs/68645/si2302cds.pdf"
-			(at 93.98 71.12 0)
+		(property "Description" "Si2302CDS-T1-GE3"
+			(at 96.52 71.12 0)
 			(hide yes)
 			(show_name no)
@@
 			)
 		)
-		(property "Description" "MOSFETs 20V Vds 8V Vgs SOT-23"
-			(at 93.98 71.12 0)
+		(property "MPN" "Si2302CDS-T1-GE3"
+			(at 96.52 91.44 0)
 			(hide yes)
 			(show_name no)
@@
 			)
 		)
-		(property "MPN" "SI2302CDS-T1-GE3 "
-			(at 93.218 67.31 0)
+		(property "Manufacturer" "VISHAY(威世)"
+			(at 96.52 88.9 0)
 			(hide yes)
 			(show_name no)
@@
 			(effects
 				(font
-					(size 0.508 0.508)
+					(size 1.27 1.27)
 				)
 			)
 		)
-		(property "Manufacturer" "Vishay"
-			(at 93.98 71.12 0)
+		(property "LCSC Part" "C10488"
+			(at 96.52 93.98 0)
 			(hide yes)
 			(show_name no)
@@
 		(on_board yes)
 		(in_pos_files yes)
-		(dnp no)
+		(dnp yes)
 		(fields_autoplaced yes)
 		(property "Reference" "BAT-1"
